File: MacroGamePad/MacroGamePad.kicad_sch (KiCad schematic)
At the start: 14 parts, among them SW1 SW_Push, SW2 SW_Push, SW3 SW_Push, SW4 SW_Push, SW5 SW_Push, SW6 RotaryEncoder_Switch, U1 MOUDLE-SEEEDUINO-XIAO

Commit message: Added pcb
Parts:
- SW6: symbol Device:RotaryEncoder_Switch -> Device:RotaryEncoder_Switch_MP
Connections:
- no-connect marks 0 -> 2
Changed lines of the file:
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@@
 		(color 0 0 0 0)
+	)
+	(no_connect
+		(at 62.23 86.36)
+	)
+	(no_connect
+		(at 104.14 78.74)
 	)
 	(wire
@@
 	(rectangle
 		(start 46.99 57.15)
-		(end 116.84 96.52)
+		(end 119.38 96.52)
 		(stroke
 			(width 0)
@@
 	)
 	(symbol
-		(lib_id "Device:RotaryEncoder_Switch")
+		(lib_id "Device:RotaryEncoder_Switch_MP")
 		(at 119.38 30.48 180)
 		(unit 1)
@@
 		(fields_autoplaced yes)
 		(property "Reference" "SW6"
-			(at 119.38 20.32 0)
+			(at 119.38 38.1 0)
 			(effects
 				(font
@@
 		)
 		(property "Value" "RotaryEncoder_Switch"
-			(at 119.38 22.86 0)
+			(at 119.38 40.64 0)
 			(effects
 				(font
@@
 		)
 		(property "Datasheet" "~"
-			(at 119.38 37.084 0)
-			(effects
-				(font
-					(size 1.27 1.27)
-				)
-				(hide yes)
-			)
-		)
-		(property "Description" "Rotary encoder, dual channel, incremental quadrate outputs, with switch"
-			(at 119.38 30.48 0)
+			(at 119.38 17.78 0)
+			(effects
+				(font
+					(size 1.27 1.27)
+				)
+				(hide yes)
+			)
+		)
+		(property "Description" "Rotary encoder, dual channel, incremental quadrate outputs, with switch and MP Pin"
+			(at 119.38 15.24 0)
 			(effects
 				(font
@@
 		(pin "S2"
 		)
+		(pin "MP"
+		)
 		(instances

Commit message: PCB finished
Connections:
- net Row 1: now also U1.11 (PA6_A10_D10_MOSI); no longer U1.2 (PA4_A1_D1)
- no-connect marks 2 -> 3
Changed lines of the file:
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@@
+	)
+	(no_connect
+		(at 119.38 22.86)
 	)
 	(no_connect
@@
 	)
 	(no_connect
-		(at 104.14 78.74)
+		(at 63.5 73.66)
 	)
 	(wire
@@
 	(global_label "Row 1"
 		(shape input)
-		(at 63.5 73.66 180)
-		(fields_autoplaced yes)
-		(effects
-			(font
-				(size 1.27 1.27)
-			)
-			(justify right)
-		)
-		(property "Intersheetrefs" "${INTERSHEET_REFS}"
-			(at 54.5882 73.66 0)
-			(effects
-				(font
-					(size 1.27 1.27)
-				)
-				(justify right)
-				(hide yes)
-			)
+		(at 104.14 78.74 0)
+		(fields_autoplaced yes)
+		(effects
+			(font
+				(size 1.27 1.27)
+			)
+			(justify left)
+		)
+		(property "Intersheetrefs" "${INTERSHEET_REFS}"
+			(at 113.0518 78.74 0)
+			(effects
+				(font
+					(size 1.27 1.27)
+				)
+				(justify left)
+				(hide yes)
+			)
